File: stlink-v3minie-uart.kicad_pcb (KiCad board)
At the start: 2 copper layers, 14 x 23 mm, 3 parts, among them J1 Conn_01x05, J2 Conn_02x05_Top_Bottom, J3 Conn_01x04_Pin

Commit message: pcb(silk): add jlcjlcjlc
Routing:
- net GND: vias 17 -> 18
Other:
- board text added: "JLCJLCJLCJLC"
- board text added: "edition"
- board text added: "君セン"
Changed lines of the file:
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@@
+		)
+	)
+	(gr_text "JLCJLCJLCJLC"
+		(at 154.864348 101.674818 0)
+		(layer "B.SilkS")
+		(effects
+			(font
+				(size 1 1)
+				(thickness 0.1)
+			)
+			(justify left bottom mirror)
+		)
+	)
+	(gr_text "edition"
+		(at 149.5 111 0)
+		(layer "B.SilkS")
+		(effects
+			(font
+				(size 1 1)
+				(thickness 0.1875)
+			)
+			(justify left bottom mirror)
 		)
 	)
@@
 		)
 	)
+	(gr_text "君セン"
+		(at 155.75 111 0)
+		(layer "B.SilkS")
+		(effects
+			(font
+				(face "Noto Sans CJK JP")
+				(size 1.3 1.3)
+				(thickness 0.1875)
+			)
+			(justify left bottom mirror)
+		)
+		(render_cache "君セン" 0
+			(polygon
+				(pts
+					(xy 155.458838 109.453054) (xy 154.989311 109.453054) (xy 155.03297 109.646103) (xy 155.651728 109.646103)
+					(xy 155.651728 109.769935) (xy 155.071151 109.769935) (xy 155.108519 109.871927) (xy 155.151244 109.969811)
+					(xy 155.480667 109.969811) (xy 155.480667 110.088085) (xy 155.21316 110.088085) (xy 155.259208 110.159559)
+					(xy 155.309715 110.227896) (xy 155.361238 110.288766) (xy 155.417129 110.34649) (xy 155.474668 110.398399)
+					(xy 155.536575 110.447106) (xy 155.600881 110.491069) (xy 155.669645 110.531719) (xy 155.686338 110.540704)
+					(xy 155.632295 110.60259) (xy 155.598941 110.650406) (xy 155.528383 110.608591) (xy 155.461963 110.563442)
+					(xy 155.340047 110.46258) (xy 155.269598 110.390757) (xy 155.269598 110.930137) (xy 155.131241 110.930137)
+					(xy 155.131241 110.840042) (xy 154.319512 110.840042) (xy 154.319512 110.926486) (xy 154.175757 110.926486)
+					(xy 154.175757 110.718036) (xy 154.319512 110.718036) (xy 155.131241 110.718036) (xy 155.131241 110.39806)
+					(xy 154.319512 110.39806) (xy 154.319512 110.718036) (xy 154.175757 110.718036) (xy 154.175757 110.276055)
+					(xy 155.174899 110.276055) (xy 155.088664 110.142745) (xy 155.05845 110.088085) (xy 154.221241 110.088085)
+					(xy 154.221241 109.969811) (xy 154.359598 109.969811) (xy 155.002012 109.969811) (xy 154.945973 109.826065)
+					(xy 154.927396 109.769935) (xy 154.359598 109.769935) (xy 154.359598 109.969811) (xy 154.221241 109.969811)
+					(xy 154.221241 109.769935) (xy 154.022873 109.769935) (xy 154.022873 109.646103) (xy 154.221241 109.646103)
+					(xy 154.359598 109.646103) (xy 154.89104 109.646103) (xy 154.843651 109.453054) (xy 154.359598 109.453054)
+					(xy 154.359598 109.646103) (xy 154.221241 109.646103) (xy 154.221241 109.332954) (xy 155.458838 109.332954)
+				)
+			)
+			(polygon
+				(pts
+					(xy 152.317575 109.732865) (xy 152.424896 109.648882) (xy 152.481564 109.671468) (xy 152.521341 109.681745)
+					(xy 153.22567 109.824071) (xy 153.22567 109.539418) (xy 153.222901 109.457711) (xy 153.213678 109.375717)
+					(xy 153.21297 109.371532) (xy 153.385857 109.371532) (xy 153.374111 109.490581) (xy 153.373156 109.539418)
+					(xy 153.373156 109.851457) (xy 153.638619 109.900285) (xy 153.820853 109.929883) (xy 153.793547 110.081418)
+					(xy 153.373156 109.993783) (xy 153.373156 110.546737) (xy 153.370273 110.606249) (xy 153.36025 110.658172)
+					(xy 153.348289 110.689205) (xy 153.331414 110.716766) (xy 153.31192 110.738219) (xy 153.287645 110.756992)
+					(xy 153.223012 110.786533) (xy 153.125801 110.806558) (xy 152.972769 110.814561) (xy 152.815589 110.812123)
+					(xy 152.672164 110.805214) (xy 152.401241 110.778206) (xy 152.393938 110.621512) (xy 152.524005 110.643575)
+					(xy 152.655162 110.659837) (xy 152.775966 110.669324) (xy 152.903052 110.673973) (xy 152.961815 110.674457)
+					(xy 153.046388 110.671778) (xy 153.111433 110.663181) (xy 153.146919 110.653074) (xy 153.174637 110.639294)
+					(xy 153.192613 110.624568) (xy 153.206134 110.606829) (xy 153.221845 110.561349) (xy 153.22567 110.508397)
+					(xy 153.22567 109.964572) (xy 152.537773 109.825897) (xy 152.617817 109.96284) (xy 152.676725 110.048202)
+					(xy 152.743425 110.134277) (xy 152.801603 110.200667) (xy 152.861718 110.260258) (xy 152.734315 110.336859)
+					(xy 152.626572 110.211545) (xy 152.503904 110.040618) (xy 152.379415 109.83825) (xy 152.361234 109.805814)
+				)
+			)
+			(polygon
+				(pts
+					(xy 151.696912 109.445989) (xy 151.80066 109.556961) (xy 151.65242 109.667882) (xy 151.437822 109.850711)
+					(xy 151.347486 109.937345) (xy 151.232783 109.822722) (xy 151.368661 109.699629) (xy 151.602929 109.512569)
+				)
+			)
+			(polygon
+				(pts
+					(xy 151.853447 110.665329) (xy 151.757001 110.814561) (xy 151.563435 110.768747) (xy 151.380727 110.706137)
+					(xy 151.20665 110.626851) (xy 151.041718 110.532528) (xy 150.893705 110.427919) (xy 150.752737 110.30442)
+					(xy 150.622843 110.164815) (xy 150.50922 110.014312) (xy 150.430183 109.884558) (xy 150.517579 109.729928)
+					(xy 150.593776 109.867553) (xy 150.643515 109.941408) (xy 150.69961 110.015502) (xy 150.761636 110.088872)
+					(xy 150.829237 110.160643) (xy 150.899401 110.227528) (xy 150.97405 110.291244) (xy 151.048069 110.347558)
+					(xy 151.125463 110.399648) (xy 151.217173 110.453266) (xy 151.319974 110.505618) (xy 151.411554 110.545749)
+					(xy 151.510985 110.582852) (xy 151.606276 110.612523) (xy 151.708183 110.638325)
+				)
+			)
+		)
+	)
 	(segment
 		(start 146 110.75)
@@
 		(size 0.9)
 		(drill 0.4)
+		(layers "F.Cu" "B.Cu")
+		(free yes)
+		(net "GND")
+	)
+	(via
+		(at 145.195694 106.155527)
+		(size 0.9)
+		(drill 0.4)
