File: stlink-v3minie-uart.kicad_sch (KiCad schematic)
At the start: 3 parts, among them J1 Conn_01x05, J2 Conn_02x05_Top_Bottom, J3 Conn_01x04_Pin

Commit message: schem/pcb: fix pin numbering
Connections:
- net +3V3: now also J2.5 (Pin_5); no longer J2.10 (Pin_10)
- net GND: now also J2.1 (Pin_1); no longer J2.6 (Pin_6)
- net JTDI: now also J2.7 (Pin_7); no longer J2.2 (Pin_2)
- net SWCLK: now also J2.9 (Pin_9); no longer J2.4 (Pin_4)
- net SWDIO: now also J2.8 (Pin_8); no longer J2.3 (Pin_3)
- net SWO: now also J2.10 (Pin_10); no longer J2.5 (Pin_5)
- net VCP_RX: now also J2.2 (Pin_2); no longer J2.7 (Pin_7)
- net VCP_TX: now also J2.3 (Pin_3); no longer J2.8 (Pin_8)
- net nRST: now also J2.4 (Pin_4); no longer J2.9 (Pin_9)
Other:
- moved on the sheet: J2
Changed lines of the file:
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@@
 	(symbol
 		(lib_id "Connector_Generic:Conn_02x05_Top_Bottom")
-		(at 138.43 104.14 0)
-		(mirror x)
+		(at 140.97 104.14 180)
 		(unit 1)
 		(body_style 1)
@@
 		(dnp no)
 		(property "Reference" "J2"
-			(at 133.604 93.98 0)
+			(at 145.796 93.98 0)
 			(show_name no)
 			(do_not_autoplace no)
@@
 		)
 		(property "Footprint" "GLCS:KYOCERA_AVX9159-006"
-			(at 138.43 104.14 0)
+			(at 140.97 104.14 0)
 			(hide yes)
 			(show_name no)
@@
 		)
 		(property "Datasheet" ""
-			(at 138.43 104.14 0)
+			(at 140.97 104.14 0)
 			(hide yes)
 			(show_name no)
@@
 		)
 		(property "Description" "Generic connector, double row, 02x05, top/bottom pin numbering scheme (row 1: 1...pins_per_row, row2: pins_per_row+1 ... num_pins), script generated (kicad-library-utils/schlib/autogen/connector/)"
-			(at 138.43 104.14 0)
+			(at 140.97 104.14 0)
 			(hide yes)
 			(show_name no)
